Commit message: Update drone_urdf2.urdf

File: urdf/drone_urdf2.urdf (robot description, URDF)
Before this commit: robot drone_urdf2, 7 links, 6 joints
Links:
- removed link Link_1
- removed link Link_2
- removed link Link_3
- removed link Link_4
- removed link Link_5
- removed link Link_6
- added link link_1, mass 0.0117525934249256; collision mesh filename=package://drone_urdf2/meshes/Link_1.STL; visual mesh filename=package://drone_urdf2/meshes/Link_1.STL
- added link link_2, mass 0.185605397053264; collision mesh filename=package://drone_urdf2/meshes/Link_2.STL; visual mesh filename=package://drone_urdf2/meshes/Link_2.STL
- added link link_3, mass 0.185605390675731; collision mesh filename=package://drone_urdf2/meshes/Link_3.STL; visual mesh filename=package://drone_urdf2/meshes/Link_3.STL
- added link link_4, mass 0.0117525934325749; collision mesh filename=package://drone_urdf2/meshes/Link_4.STL; visual mesh filename=package://drone_urdf2/meshes/Link_4.STL
- added link link_5, mass 0.185605351162656; collision mesh filename=package://drone_urdf2/meshes/Link_5.STL; visual mesh filename=package://drone_urdf2/meshes/Link_5.STL
- added link link_6, mass 0.185604947450906; collision mesh filename=package://drone_urdf2/meshes/Link_6.STL; visual mesh filename=package://drone_urdf2/meshes/Link_6.STL
- added link world
Joints:
- added joint base_joint: type fixed, parent world, child base_link, origin xyz=0.0 0.0 0.0 rpy=0 0 3.142
- joint joint_5: child Link_5 -> link_5; parent Link_4 -> link_4
- joint joint_6: child Link_6 -> link_6; parent Link_4 -> link_4
